File: pcb/switches.sch (KiCad schematic (older format))
At the start: 84 parts

Commit message: added switches and diodes
Parts:
- added D_0, D_1, D_2, D_3, D_4, D_5, D_6, D_7, D_8, D_9, D_A, D_B, D_BACKSPACE, D_BSLSH, D_C, D_CAPS, D_COMMA, D_D, D_DELETE, D_DOT, D_DOWN, D_E, D_END, D_ENTER, D_EQUALS, D_ESC, D_F, D_F1, D_F10, D_F11, D_F12, D_F2, D_F3, D_F4, D_F5, D_F6, D_F7, D_F8, D_F9, D_FN, D_G, D_H, D_HOME, D_I, D_J, D_K, D_L, D_LALT, D_LBRAC, D_LCTRL, D_LEFT, D_LSHIFT, D_M, D_MINUS, D_N, D_O, D_OS, D_P, D_PAUSE, D_PGDN, D_PGUP, D_PRTSC, D_Q, D_QUOTE, D_R, D_RALT, D_RBRAC, D_RCTRL, D_RIGHT, D_RSHIFT, D_S, D_SEMIC, D_SLASH, D_SPACE, D_T, D_TAB, D_TILDE, D_U, D_UP, D_V, D_W, D_X, D_Y, D_Z: D, symbol Device:D

Commit message: connected rows and columns
Connections:
- net col0: now reaches K_ESC.1
- net col0: now also K_CAPS.1, K_LCTRL.1, K_TAB.1, K_TILDE.1
- net at K_ESC.2: now also D_ESC.2 (A)
- net col1: now reaches K_F1.1
- net col1: now also K_1.1, K_LSHIFT.1, K_OS.1
- net at K_F1.2: now also D_F1.2 (A)
- net col2: now reaches K_F2.1
- net col2: now also K_2.1, K_A.1, K_Q.1, K_Z.1
- net at K_F2.2: now also D_F2.2 (A)
- net col3: now reaches K_F3.1
- net col3: now also K_3.1, K_LALT.1, K_S.1, K_W.1, K_X.1
- net at K_F3.2: now also D_F3.2 (A)
- net col4: now reaches K_F4.1
- net col4: now also K_4.1, K_C.1, K_D.1, K_E.1
- net at K_F4.2: now also D_F4.2 (A)
- net col5: now reaches K_F5.1
- net col5: now also K_5.1, K_F.1, K_R.1, K_V.1
- net at K_F5.2: now also D_F5.2 (A)
- net col6: now reaches K_F6.1
- net col6: now also K_6.1, K_B.1, K_G.1, K_SPACE.1, K_T.1
- net at K_F6.2: now also D_F6.2 (A)
- net col7: now reaches K_F7.1
- net col7: now also K_7.1, K_H.1, K_N.1, K_Y.1
- net at K_F7.2: now also D_F7.2 (A)
- net col8: now reaches K_F8.1
- net col8: now also K_8.1, K_J.1, K_M.1, K_U.1
- net at K_F8.2: now also D_F8.2 (A)
- net col9: now reaches K_F9.1
- net col9: now also K_9.1, K_COMMA.1, K_I.1, K_K.1
- net at K_F9.2: now also D_F9.2 (A)
- net col10: now reaches K_F10.1
- net col10: now also K_0.1, K_DOT.1, K_L.1, K_O.1, K_RALT.1
- net at K_F10.2: now also D_F10.2 (A)
- net col11: now reaches K_F11.1
- net col11: now also K_FN.1, K_MINUS.1, K_P.1, K_SEMIC.1, K_SLASH.1
- net at K_F11.2: now also D_F11.2 (A)
- net col12: now reaches K_F12.1
- net col12: now also K_EQUALS.1, K_LBRAC.1, K_QUOTE.1, K_RCTRL.1
- net at K_F12.2: now also D_F12.2 (A)
- net col13: now reaches K_PRTSC.1
- net col13: now also K_ENTER.1, K_LEFT.1, K_RBRAC.1, K_RSHIFT.1
- net at K_PRTSC.2: now also D_PRTSC.2 (A)
- net col14: now reaches K_PAUSE.1
- net col14: now also K_BACKSPACE.1, K_BSLSH.1, K_DOWN.1, K_UP.1
- net at K_PAUSE.2: now also D_PAUSE.2 (A)
- net col15: now reaches K_DELETE.1
- net col15: now also K_END.1, K_HOME.1, K_PGDN.1, K_PGUP.1, K_RIGHT.1
- net at K_DELETE.2: now also D_DELETE.2 (A)
- net at K_TILDE.2: now also D_TILDE.2 (A)
- net at K_1.2: now also D_1.2 (A)
- net at K_2.2: now also D_2.2 (A)
- net at K_3.2: now also D_3.2 (A)
- net at K_4.2: now also D_4.2 (A)
- net at K_5.2: now also D_5.2 (A)
- net at K_6.2: now also D_6.2 (A)
- net at K_7.2: now also D_7.2 (A)
- net at K_8.2: now also D_8.2 (A)
- net at K_9.2: now also D_9.2 (A)
- net at K_0.2: now also D_0.2 (A)
- net at K_MINUS.2: now also D_MINUS.2 (A)
- net at K_EQUALS.2: now also D_EQUALS.2 (A)
- net at K_BACKSPACE.2: now also D_BACKSPACE.2 (A)
- net at K_HOME.2: now also D_HOME.2 (A)
- net at K_TAB.2: now also D_TAB.2 (A)
- net at K_Q.2: now also D_Q.2 (A)
- net at K_W.2: now also D_W.2 (A)
- net at K_E.2: now also D_E.2 (A)
- net at K_R.2: now also D_R.2 (A)
- net at K_T.2: now also D_T.2 (A)
- net at K_Y.2: now also D_Y.2 (A)
- net at K_U.2: now also D_U.2 (A)
- net at K_I.2: now also D_I.2 (A)
- net at K_O.2: now also D_O.2 (A)
- net at K_P.2: now also D_P.2 (A)
- net at K_LBRAC.2: now also D_LBRAC.2 (A)
- net at K_RBRAC.2: now also D_RBRAC.2 (A)
- net at K_BSLSH.2: now also D_BSLSH.2 (A)
- net at K_PGUP.2: now also D_PGUP.2 (A)
- net at K_CAPS.2: now also D_CAPS.2 (A)
- net at K_A.2: now also D_A.2 (A)
- net at K_S.2: now also D_S.2 (A)
- net at K_D.2: now also D_D.2 (A)
- net at K_F.2: now also D_F.2 (A)
- net at K_H.2: now also D_H.2 (A)
- net at K_J.2: now also D_J.2 (A)
- net at K_K.2: now also D_K.2 (A)
- net at K_L.2: now also D_L.2 (A)
- net at K_SEMIC.2: now also D_SEMIC.2 (A)
- net at K_QUOTE.2: now also D_QUOTE.2 (A)
- net at K_ENTER.2: now also D_ENTER.2 (A)
- net at K_PGDN.2: now also D_PGDN.2 (A)
- net at K_G.2: now also D_G.2 (A)
- net at K_LSHIFT.2: now also D_LSHIFT.2 (A)
- net at K_Z.2: now also D_Z.2 (A)
- net at K_X.2: now also D_X.2 (A)
- net at K_C.2: now also D_C.2 (A)
- net at K_V.2: now also D_V.2 (A)
- net at K_N.2: now also D_N.2 (A)
- net at K_M.2: now also D_M.2 (A)
- net at K_COMMA.2: now also D_COMMA.2 (A)
- net at K_DOT.2: now also D_DOT.2 (A)
- net at K_SLASH.2: now also D_SLASH.2 (A)
- net at K_RSHIFT.2: now also D_RSHIFT.2 (A)
- net at K_UP.2: now also D_UP.2 (A)
- net at K_END.2: now also D_END.2 (A)
- net at K_B.2: now also D_B.2 (A)
- net at K_LCTRL.2: now also D_LCTRL.2 (A)
- net at K_OS.2: now also D_OS.2 (A)
- net at K_LALT.2: now also D_LALT.2 (A)
- net at K_SPACE.2: now also D_SPACE.2 (A)
- net at K_RALT.2: now also D_RALT.2 (A)
- net at K_FN.2: now also D_FN.2 (A)
- net at K_RCTRL.2: now also D_RCTRL.2 (A)
- net at K_DOWN.2: now also D_DOWN.2 (A)
- net at K_RIGHT.2: now also D_RIGHT.2 (A)
- net at K_LEFT.2: now also D_LEFT.2 (A)
- net row0: now reaches D_ESC.1 (K)
- net row0: now also D_DELETE.1 (K), D_F1.1 (K), D_F10.1 (K), D_F11.1 (K), D_F12.1 (K), D_F2.1 (K), D_F3.1 (K), D_F4.1 (K), D_F5.1 (K), D_F6.1 (K), D_F7.1 (K), D_F8.1 (K), D_F9.1 (K), D_PAUSE.1 (K), D_PRTSC.1 (K)
- net row1: now reaches D_TILDE.1 (K)
- net row1: now also D_0.1 (K), D_1.1 (K), D_2.1 (K), D_3.1 (K), D_4.1 (K), D_5.1 (K), D_6.1 (K), D_7.1 (K), D_8.1 (K), D_9.1 (K), D_BACKSPACE.1 (K), D_EQUALS.1 (K), D_HOME.1 (K), D_MINUS.1 (K)
- net row2: now reaches D_TAB.1 (K)
- net row2: now also D_BSLSH.1 (K), D_E.1 (K), D_I.1 (K), D_LBRAC.1 (K), D_O.1 (K), D_P.1 (K), D_PGUP.1 (K), D_Q.1 (K), D_R.1 (K), D_RBRAC.1 (K), D_T.1 (K), D_U.1 (K), D_W.1 (K), D_Y.1 (K)
- net row3: now reaches D_CAPS.1 (K)
- net row3: now also D_A.1 (K), D_D.1 (K), D_ENTER.1 (K), D_F.1 (K), D_G.1 (K), D_H.1 (K), D_J.1 (K), D_K.1 (K), D_L.1 (K), D_PGDN.1 (K), D_QUOTE.1 (K), D_S.1 (K), D_SEMIC.1 (K)
- net row4: now reaches D_LSHIFT.1 (K)
- net row4: now also D_B.1 (K), D_C.1 (K), D_COMMA.1 (K), D_DOT.1 (K), D_END.1 (K), D_M.1 (K), D_N.1 (K), D_RSHIFT.1 (K), D_SLASH.1 (K), D_UP.1 (K), D_V.1 (K), D_X.1 (K), D_Z.1 (K)
- net row5: now reaches D_LCTRL.1 (K)
- net row5: now also D_DOWN.1 (K), D_FN.1 (K), D_LALT.1 (K), D_LEFT.1 (K), D_OS.1 (K), D_RALT.1 (K), D_RCTRL.1 (K), D_RIGHT.1 (K), D_SPACE.1 (K)

Commit message: why does kicad need numbered annotation? ugh
Parts:
- D_0, D_1, D_2, D_3, D_4, D_5, D_6, D_7, D_8, D_9, D_A, D_B, D_BACKSPACE, D_BSLSH, D_C, D_CAPS, D_COMMA, D_D, D_DELETE, D_DOT, D_DOWN, D_E, D_END, D_ENTER, D_EQUALS, D_ESC, D_F, D_F1, D_F10, D_F11, D_F12, D_F2, D_F3, D_F4, D_F5, D_F6, D_F7, D_F8, D_F9, D_FN, D_G, D_H, D_HOME, D_I, D_J, D_K, D_L, D_LALT, D_LBRAC, D_LCTRL, D_LEFT, D_LSHIFT, D_M, D_MINUS, D_N, D_O, D_OS, D_P, D_PAUSE, D_PGDN, D_PGUP, D_PRTSC, D_Q, D_QUOTE, D_R, D_RALT, D_RBRAC, D_RCTRL, D_RIGHT, D_RSHIFT, D_S, D_SEMIC, D_SLASH, D_SPACE, D_T, D_TAB, D_TILDE, D_U, D_UP, D_V, D_W, D_X, D_Y, D_Z: footprint (none) -> parts:D_SOD123_axial

Commit message: added number to annotations
Parts:
- renumbered D_0 to D_0_1, D_1 to D_1_1, D_2 to D_2_1, D_3 to D_3_1, D_4 to D_4_1, D_5 to D_5_1, D_6 to D_6_1, D_7 to D_7_1, D_8 to D_8_1, D_9 to D_9_1, D_A to D_A_1, D_BACKSPACE to D_BKSPACE_1, D_BSLSH to D_BSLSH_1, D_B to D_B_1, D_CAPS to D_CAPS_1, D_COMMA to D_COMMA_1, D_C to D_C_1, D_DELETE to D_DELETE_1, D_DOT to D_DOT_1, D_DOWN to D_DOWN_1, D_D to D_D_1, D_END to D_END_1, D_ENTER to D_ENTER_1, D_EQUALS to D_EQUALS_1, D_ESC to D_ESC_1, D_E to D_E_1, D_F10 to D_F10_1, D_F11 to D_F11_1, D_F12 to D_F12_1, D_F1 to D_F1_1, D_F2 to D_F2_1, D_F3 to D_F3_1, D_F4 to D_F4_1, D_F5 to D_F5_1, D_F6 to D_F6_1, D_F7 to D_F7_1, D_F8 to D_F8_1, D_F9 to D_F9_1, D_FN to D_FN_1, D_F to D_F_1, D_G to D_G_1, D_HOME to D_HOME_1, D_H to D_H_1, D_I to D_I_1, D_J to D_J_1, D_K to D_K_1, D_LALT to D_LALT_1, D_LBRAC to D_LBRAC_1, D_LCTRL to D_LCTRL_1, D_LEFT to D_LEFT_1, D_LSHIFT to D_LSHIFT_1, D_L to D_L_1, D_MINUS to D_MINUS_1, D_M to D_M_1, D_N to D_N_1, D_OS to D_OS_1, D_O to D_O_1, D_PAUSE to D_PAUSE_1, D_PGDN to D_PGDN_1, D_PGUP to D_PGUP_1, D_PRTSC to D_PRTSC_1, D_P to D_P_1, D_QUOTE to D_QUOTE_1, D_Q to D_Q_1, D_RALT to D_RALT_1, D_RBRAC to D_RBRAC_1, D_RCTRL to D_RCTRL_1, D_RIGHT to D_RIGHT_1, D_RSHIFT to D_RSHIFT_1, D_R to D_R_1, D_SEMIC to D_SEMIC_1, D_SLASH to D_SLASH_1, D_SPACE to D_SPACE_1, D_S to D_S_1, D_TAB to D_TAB_1, D_TILDE to D_TILDE_1, D_T to D_T_1, D_UP to D_UP_1, D_U to D_U_1, D_V to D_V_1, D_W to D_W_1, D_X to D_X_1, D_Y to D_Y_1, D_Z to D_Z_1, K_0 to K_0_1, K_1 to K_1_1, K_2 to K_2_1, K_3 to K_3_1, K_4 to K_4_1, K_5 to K_5_1, K_6 to K_6_1, K_7 to K_7_1, K_8 to K_8_1, K_9 to K_9_1, K_A to K_A_1, K_BACKSPACE to K_BKSPACE_1, K_BSLSH to K_BSLSH_1, K_B to K_B_1, K_CAPS to K_CAPS_1, K_COMMA to K_COMMA_1, K_C to K_C_1, K_DELETE to K_DELETE_1, K_DOT to K_DOT_1, K_DOWN to K_DOWN_1, K_D to K_D_1, K_END to K_END_1, K_ENTER to K_ENTER_1, K_EQUALS to K_EQUALS_1, K_ESC to K_ESC_1, K_E to K_E_1, K_F10 to K_F10_1, K_F11 to K_F11_1, K_F12 to K_F12_1, K_F1 to K_F1_1, K_F2 to K_F2_1, K_F3 to K_F3_1, K_F4 to K_F4_1, K_F5 to K_F5_1, K_F6 to K_F6_1, K_F7 to K_F7_1, K_F8 to K_F8_1, K_F9 to K_F9_1, K_FN to K_FN_1, K_F to K_F_1, K_G to K_G_1, K_HOME to K_HOME_1, K_H to K_H_1, K_I to K_I_1, K_J to K_J_1, K_K to K_K_1, K_LALT to K_LALT_1, K_LBRAC to K_LBRAC_1, K_LCTRL to K_LCTRL_1, K_LEFT to K_LEFT_1, K_LSHIFT to K_LSHIFT_1, K_L to K_L_1, K_MINUS to K_MINUS_1, K_M to K_M_1, K_N to K_N_1, K_OS to K_OS_1, K_O to K_O_1, K_PAUSE to K_PAUSE_1, K_PGDN to K_PGDN_1, K_PGUP to K_PGUP_1, K_PRTSC to K_PRTSC_1, K_P to K_P_1, K_QUOTE to K_QUOTE_1, K_Q to K_Q_1, K_RALT to K_RALT_1, K_RBRAC to K_RBRAC_1, K_RCTRL to K_RCTRL_1, K_RIGHT to K_RIGHT_1, K_RSHIFT to K_RSHIFT_1, K_R to K_R_1, K_SEMIC to K_SEMIC_1, K_SLASH to K_SLASH_1, K_SPACE to K_SPACE_1, K_S to K_S_1, K_TAB to K_TAB_1, K_TILDE to K_TILDE_1, K_T to K_T_1, K_UP to K_UP_1, K_U to K_U_1, K_V to K_V_1, K_W to K_W_1, K_X to K_X_1, K_Y to K_Y_1, K_Z to K_Z_1

Commit message: replaced with MX switches
Parts:
- removed K_0_1, K_1_1, K_2_1, K_3_1, K_4_1, K_5_1, K_6_1, K_7_1, K_8_1, K_9_1, K_A_1, K_BKSPACE_1, K_BSLSH_1, K_B_1, K_CAPS_1, K_COMMA_1, K_C_1, K_DELETE_1, K_DOT_1, K_DOWN_1, K_D_1, K_END_1, K_ENTER_1, K_EQUALS_1, K_ESC_1, K_E_1, K_F10_1, K_F11_1, K_F12_1, K_F1_1, K_F2_1, K_F3_1, K_F4_1, K_F5_1, K_F6_1, K_F7_1, K_F8_1, K_F9_1, K_FN_1, K_F_1, K_G_1, K_HOME_1, K_H_1, K_I_1, K_J_1, K_K_1, K_LALT_1, K_LBRAC_1, K_LCTRL_1, K_LEFT_1, K_LSHIFT_1, K_L_1, K_MINUS_1, K_M_1, K_N_1, K_OS_1, K_O_1, K_PAUSE_1, K_PGDN_1, K_PGUP_1, K_PRTSC_1, K_P_1, K_QUOTE_1, K_Q_1, K_RALT_1, K_RBRAC_1, K_RCTRL_1, K_RIGHT_1, K_RSHIFT_1, K_R_1, K_SEMIC_1, K_SLASH_1, K_SPACE_1, K_S_1, K_TAB_1, K_TILDE_1, K_T_1, K_UP_1, K_U_1, K_V_1, K_W_1, K_X_1, K_Y_1, K_Z_1: KEYSW, symbol parts:KEYSW
- added MX_0_1, MX_1_1, MX_2_1, MX_3_1, MX_4_1, MX_5_1, MX_6_1, MX_7_1, MX_8_1, MX_9_1, MX_A_1, MX_BKSPACE_1, MX_BSLSH_1, MX_B_1, MX_CAPS_1, MX_COMMA_1, MX_C_1, MX_DELETE_1, MX_DOT_1, MX_DOWN_1, MX_D_1, MX_END_1, MX_ENTER_1, MX_EQUALS_1, MX_ESC_1, MX_E_1, MX_F10_1, MX_F11_1, MX_F12_1, MX_F1_1, MX_F2_1, MX_F3_1, MX_F4_1, MX_F5_1, MX_F6_1, MX_F7_1, MX_F8_1, MX_F9_1, MX_FN_1, MX_F_1, MX_G_1, MX_HOME_1, MX_H_1, MX_I_1, MX_J_1, MX_K_1, MX_LALT_1, MX_LBRAC_1, MX_LCTRL_1, MX_LEFT_1, MX_LSHIFT_1, MX_L_1, MX_MINUS_1, MX_M_1, MX_N_1, MX_OS_1, MX_O_1, MX_PAUSE_1, MX_PGDN_1, MX_PGUP_1, MX_PRTSC_1, MX_P_1, MX_QUOTE_1, MX_Q_1, MX_RALT_1, MX_RBRAC_1, MX_RCTRL_1, MX_RIGHT_1, MX_RSHIFT_1, MX_R_1, MX_SEMIC_1, MX_SLASH_1, MX_SPACE_1, MX_S_1, MX_TAB_1, MX_TILDE_1, MX_T_1, MX_UP_1, MX_U_1, MX_V_1, MX_W_1, MX_X_1, MX_Y_1, MX_Z_1: MX-LED, symbol keys:MX-LED
Connections:
- net col0: now also MX_CAPS_1.1 (COL), MX_ESC_1.1 (COL), MX_LCTRL_1.1 (COL), MX_TAB_1.1 (COL), MX_TILDE_1.1 (COL)
- net col1: now also MX_1_1.1 (COL), MX_F1_1.1 (COL), MX_LSHIFT_1.1 (COL), MX_OS_1.1 (COL)
- net col10: now also MX_0_1.1 (COL), MX_DOT_1.1 (COL), MX_F10_1.1 (COL), MX_L_1.1 (COL), MX_O_1.1 (COL), MX_RALT_1.1 (COL)
- net col11: now also MX_F11_1.1 (COL), MX_FN_1.1 (COL), MX_MINUS_1.1 (COL), MX_P_1.1 (COL), MX_SEMIC_1.1 (COL), MX_SLASH_1.1 (COL)
- net col12: now also MX_EQUALS_1.1 (COL), MX_F12_1.1 (COL), MX_LBRAC_1.1 (COL), MX_QUOTE_1.1 (COL), MX_RCTRL_1.1 (COL)
- net col13: now also MX_ENTER_1.1 (COL), MX_LEFT_1.1 (COL), MX_PRTSC_1.1 (COL), MX_RBRAC_1.1 (COL), MX_RSHIFT_1.1 (COL)
- net col14: now also MX_BKSPACE_1.1 (COL), MX_BSLSH_1.1 (COL), MX_DOWN_1.1 (COL), MX_PAUSE_1.1 (COL), MX_UP_1.1 (COL)
- net col15: now also MX_DELETE_1.1 (COL), MX_END_1.1 (COL), MX_HOME_1.1 (COL), MX_PGDN_1.1 (COL), MX_PGUP_1.1 (COL), MX_RIGHT_1.1 (COL)
- net col2: now also MX_2_1.1 (COL), MX_A_1.1 (COL), MX_F2_1.1 (COL), MX_Q_1.1 (COL), MX_Z_1.1 (COL)
- net col3: now also MX_3_1.1 (COL), MX_F3_1.1 (COL), MX_LALT_1.1 (COL), MX_S_1.1 (COL), MX_W_1.1 (COL), MX_X_1.1 (COL)
- net col4: now also MX_4_1.1 (COL), MX_C_1.1 (COL), MX_D_1.1 (COL), MX_E_1.1 (COL), MX_F4_1.1 (COL)
- net col5: now also MX_5_1.1 (COL), MX_F5_1.1 (COL), MX_F_1.1 (COL), MX_R_1.1 (COL), MX_V_1.1 (COL)
- net col6: now also MX_6_1.1 (COL), MX_B_1.1 (COL), MX_F6_1.1 (COL), MX_G_1.1 (COL), MX_SPACE_1.1 (COL), MX_T_1.1 (COL)
- net col7: now also MX_7_1.1 (COL), MX_H_1.1 (COL), MX_N_1.1 (COL), MX_Y_1.1 (COL)
- net col8: now also MX_8_1.1 (COL), MX_F8_1.1 (COL), MX_J_1.1 (COL), MX_M_1.1 (COL), MX_U_1.1 (COL)
- net col9: now also MX_9_1.1 (COL), MX_COMMA_1.1 (COL), MX_F9_1.1 (COL), MX_I_1.1 (COL), MX_K_1.1 (COL)
- net at D_ESC_1.2 (A): now also MX_ESC_1.2 (ROW)
- net at D_F1_1.2 (A): now also MX_F1_1.2 (ROW)
- net at D_F2_1.2 (A): now also MX_F2_1.2 (ROW)
- net at D_F3_1.2 (A): now also MX_F3_1.2 (ROW)
- net at D_F4_1.2 (A): now also MX_F4_1.2 (ROW)
- net at D_F5_1.2 (A): now also MX_F5_1.2 (ROW)
- net at D_F6_1.2 (A): now also MX_F6_1.2 (ROW)
- net at D_F7_1.2 (A): now also MX_F7_1.2 (ROW)
- net at D_F8_1.2 (A): now also MX_F8_1.2 (ROW)
- net at D_F9_1.2 (A): now also MX_F9_1.2 (ROW)
- net at D_F10_1.2 (A): now also MX_F10_1.2 (ROW)
- net at D_F11_1.2 (A): now also MX_F11_1.2 (ROW)
- net at D_F12_1.2 (A): now also MX_F12_1.2 (ROW)
- net at D_PRTSC_1.2 (A): now also MX_PRTSC_1.2 (ROW)
- net at D_PAUSE_1.2 (A): now also MX_PAUSE_1.2 (ROW)
- net at D_DELETE_1.2 (A): now also MX_DELETE_1.2 (ROW)
- net at D_TILDE_1.2 (A): now also MX_TILDE_1.2 (ROW)
- net at D_1_1.2 (A): now also MX_1_1.2 (ROW)
- net at D_2_1.2 (A): now also MX_2_1.2 (ROW)
- net at D_3_1.2 (A): now also MX_3_1.2 (ROW)
- net at D_4_1.2 (A): now also MX_4_1.2 (ROW)
- net at D_5_1.2 (A): now also MX_5_1.2 (ROW)
- net at D_6_1.2 (A): now also MX_6_1.2 (ROW)
- net at D_7_1.2 (A): now also MX_7_1.2 (ROW)
- net at D_8_1.2 (A): now also MX_8_1.2 (ROW)
- net at D_9_1.2 (A): now also MX_9_1.2 (ROW)
- net at D_0_1.2 (A): now also MX_0_1.2 (ROW)
- net at D_MINUS_1.2 (A): now also MX_MINUS_1.2 (ROW)
- net at D_EQUALS_1.2 (A): now also MX_EQUALS_1.2 (ROW)
- net at D_BKSPACE_1.2 (A): now also MX_BKSPACE_1.2 (ROW)
- net at D_HOME_1.2 (A): now also MX_HOME_1.2 (ROW)
- net at D_TAB_1.2 (A): now also MX_TAB_1.2 (ROW)
- net at D_Q_1.2 (A): now also MX_Q_1.2 (ROW)
- net at D_W_1.2 (A): now also MX_W_1.2 (ROW)
- net at D_E_1.2 (A): now also MX_E_1.2 (ROW)
- net at D_R_1.2 (A): now also MX_R_1.2 (ROW)
- net at D_T_1.2 (A): now also MX_T_1.2 (ROW)
- net at D_Y_1.2 (A): now also MX_Y_1.2 (ROW)
- net at D_U_1.2 (A): now also MX_U_1.2 (ROW)
- net at D_I_1.2 (A): now also MX_I_1.2 (ROW)
- net at D_O_1.2 (A): now also MX_O_1.2 (ROW)
- net at D_P_1.2 (A): now also MX_P_1.2 (ROW)
- net at D_LBRAC_1.2 (A): now also MX_LBRAC_1.2 (ROW)
- net at D_RBRAC_1.2 (A): now also MX_RBRAC_1.2 (ROW)
- net at D_BSLSH_1.2 (A): now also MX_BSLSH_1.2 (ROW)
- net at D_PGUP_1.2 (A): now also MX_PGUP_1.2 (ROW)
- net at D_CAPS_1.2 (A): now also MX_CAPS_1.2 (ROW)
- net at D_A_1.2 (A): now also MX_A_1.2 (ROW)
- net at D_S_1.2 (A): now also MX_S_1.2 (ROW)
- net at D_D_1.2 (A): now also MX_D_1.2 (ROW)
- net at D_F_1.2 (A): now also MX_F_1.2 (ROW)
- net at D_H_1.2 (A): now also MX_H_1.2 (ROW)
- net at D_J_1.2 (A): now also MX_J_1.2 (ROW)
- net at D_K_1.2 (A): now also MX_K_1.2 (ROW)
- net at D_L_1.2 (A): now also MX_L_1.2 (ROW)
- net at D_SEMIC_1.2 (A): now also MX_SEMIC_1.2 (ROW)
- net at D_QUOTE_1.2 (A): now also MX_QUOTE_1.2 (ROW)
- net at D_ENTER_1.2 (A): now also MX_ENTER_1.2 (ROW)
- net at D_PGDN_1.2 (A): now also MX_PGDN_1.2 (ROW)
- net at D_G_1.2 (A): now also MX_G_1.2 (ROW)
- net at D_LSHIFT_1.2 (A): now also MX_LSHIFT_1.2 (ROW)
- net at D_Z_1.2 (A): now also MX_Z_1.2 (ROW)
- net at D_X_1.2 (A): now also MX_X_1.2 (ROW)
- net at D_C_1.2 (A): now also MX_C_1.2 (ROW)
- net at D_V_1.2 (A): now also MX_V_1.2 (ROW)
- net at D_N_1.2 (A): now also MX_N_1.2 (ROW)
- net at D_M_1.2 (A): now also MX_M_1.2 (ROW)
- net at D_COMMA_1.2 (A): now also MX_COMMA_1.2 (ROW)
- net at D_DOT_1.2 (A): now also MX_DOT_1.2 (ROW)
- net at D_SLASH_1.2 (A): now also MX_SLASH_1.2 (ROW)
- net at D_RSHIFT_1.2 (A): now also MX_RSHIFT_1.2 (ROW)
- net at D_UP_1.2 (A): now also MX_UP_1.2 (ROW)
- net at D_END_1.2 (A): now also MX_END_1.2 (ROW)
- net at D_B_1.2 (A): now also MX_B_1.2 (ROW)
- net at D_LCTRL_1.2 (A): now also MX_LCTRL_1.2 (ROW)
- net at D_OS_1.2 (A): now also MX_OS_1.2 (ROW)
- net at D_LALT_1.2 (A): now also MX_LALT_1.2 (ROW)
- net at D_SPACE_1.2 (A): now also MX_SPACE_1.2 (ROW)
- net at D_RALT_1.2 (A): now also MX_RALT_1.2 (ROW)
- net at D_FN_1.2 (A): now also MX_FN_1.2 (ROW)
- net at D_RCTRL_1.2 (A): now also MX_RCTRL_1.2 (ROW)
- net at D_DOWN_1.2 (A): now also MX_DOWN_1.2 (ROW)
- net at D_RIGHT_1.2 (A): now also MX_RIGHT_1.2 (ROW)
- net at D_LEFT_1.2 (A): now also MX_LEFT_1.2 (ROW)
