File: pcb/switches.sch (KiCad schematic (older format))
At the start: 252 parts

Commit message: moving stuff around
Parts:
- renumbered D_BKSPACE_1 to D_BSPACE_1, D_DELETE_1 to D_DEL_1, MX_BKSPACE_1 to MX_BSPACE_1, MX_DELETE_1 to MX_DEL_1, R_BKSPACE_1 to R_BSPACE_1, R_DELETE_1 to R_DEL_1
Changed lines of the file:
@@
 $EndComp
 $Comp
-L Device:D D_DELETE_1
+L Device:D D_DEL_1
 U 1 1 5F76CE6A
 P 19000 5600
-F 0 "D_DELETE_1" V 19046 5520 50  0000 R CNN
+F 0 "D_DEL_1" V 19046 5520 50  0000 R CNN
 F 1 "D" V 18955 5520 50  0000 R CNN
 F 2 "parts:D_SOD123_axial" H 19000 5600 50  0001 C CNN
@@
 $EndComp
 $Comp
-L Device:D D_BKSPACE_1
+L Device:D D_BSPACE_1
 U 1 1 5F78A2D7
 P 18000 6600
-F 0 "D_BKSPACE_1" V 18046 6520 50  0000 R CNN
+F 0 "D_BSPACE_1" V 18046 6520 50  0000 R CNN
 F 1 "D" V 17955 6520 50  0000 R CNN
 F 2 "parts:D_SOD123_axial" H 18000 6600 50  0001 C CNN
@@
 $EndComp
 $Comp
-L keys:MX-LED MX_DELETE_1
+L keys:MX-LED MX_DEL_1
 U 1 1 5F7C8D70
 P 19050 5200
-F 0 "MX_DELETE_1" H 19132 5424 60  0000 C CNN
+F 0 "MX_DEL_1" H 19132 5424 60  0000 C CNN
 F 1 "MX-LED" H 19132 5350 20  0000 C CNN
 F 2 "keys:MX-1U" H 18425 5175 60  0001 C CNN
@@
 $EndComp
 $Comp
-L keys:MX-LED MX_BKSPACE_1
+L keys:MX-LED MX_BSPACE_1
 U 1 1 5F7F47BC
 P 18050 6200
-F 0 "MX_BKSPACE_1" H 18132 6424 60  0000 C CNN
+F 0 "MX_BSPACE_1" H 18132 6424 60  0000 C CNN
 F 1 "MX-LED" H 18132 6350 20  0000 C CNN
 F 2 "keys:MX-2U-ReversedStabilizers" H 17425 6175 60  0001 C CNN
@@
 $EndComp
 $Comp
-L Device:R R_DELETE_1
+L Device:R R_DEL_1
 U 1 1 611BF026
 P 19150 5350
-F 0 "R_DELETE_1" H 19220 5396 50  0000 L CNN
+F 0 "R_DEL_1" H 19220 5396 50  0000 L CNN
 F 1 "470" H 19220 5305 50  0000 L CNN
 F 2 "Resistor_THT:R_Axial_DIN0207_L6.3mm_D2.5mm_P7.62mm_Horizontal" V 19080 5350 50  0001 C CNN
@@
 $EndComp
 $Comp
-L Device:R R_BKSPACE_1
+L Device:R R_BSPACE_1
 U 1 1 611C4B6B
 P 18150 6350
-F 0 "R_BKSPACE_1" H 18220 6396 50  0000 L CNN
+F 0 "R_BSPACE_1" H 18220 6396 50  0000 L CNN
 F 1 "470" H 18220 6305 50  0000 L CNN
 F 2 "Resistor_THT:R_Axial_DIN0207_L6.3mm_D2.5mm_P7.62mm_Horizontal" V 18080 6350 50  0001 C CNN
