File: pcb/00Key.kicad_pcb (KiCad board)
At the start: 2 copper layers, 304.8 x 173.4 mm, 260 parts, among them Q1 IRLZ44N, U1 Teensy4.1

Commit message: moving stuff around
Parts:
- removed R_BKSPACE_1, R_DELETE_1: 470, Resistor_THT:R_Axial_DIN0207_L6.3mm_D2.5mm_P7.62mm_Horizontal
- added R_BSPACE_1: 470, Resistor_THT:R_Axial_DIN0207_L6.3mm_D2.5mm_P7.62mm_Horizontal, F.Cu at (292.7, 83.8)
- added R_DEL_1: 470, Resistor_THT:R_Axial_DIN0207_L6.3mm_D2.5mm_P7.62mm_Horizontal, F.Cu at (304.2, 85.7)
- moved U1 11.0 mm to (291.8, 54.9), turned to 180 degrees
- moved Q1 5.43 mm to (329.6, 76.6)
- moved R_Q1_GATE_1 5.43 mm to (328.4, 84.3)
- moved R_DOWN_1 2.85 mm to (301.3, 78.1)
- moved R_END_1 2.85 mm to (315.6, 78.1)
- moved R_ENTER_1 2.85 mm to (281.3, 81.9)
- moved R_PGDN_1 2.85 mm to (312.7, 80.0)
- moved R_RCTRL_1 2.85 mm to (272.7, 78.1)
- moved R_RSHIFT_1 2.85 mm to (284.2, 80.0)
- moved R_EQUALS_1 2.85 mm to (264.2, 83.8)
- moved R_F12_1 2.85 mm to (261.3, 85.7)
- moved R_B_1 2.85 mm to (178.4, 78.1)
- moved R_CAPS_1 2.85 mm to (89.9, 80.0)
- moved R_COMMA_1 2.85 mm to (224.2, 78.1)
- moved R_C_1 2.85 mm to (149.9, 78.1)
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- renumbered D_BKSPACE_1 to D_BSPACE_1, D_DELETE_1 to D_DEL_1, MX_BKSPACE_1 to MX_BSPACE_1, MX_DELETE_1 to MX_DEL_1
Other:
- board size 304.8 x 173.4 mm -> 304.8 x 170.8 mm

Commit message: logo
Other:
- board text added: "00Key"
- board text added: "By 001"

Commit message: holes
Parts:
- added REF**: MountingHole_2.2mm_M2_Pad, MountingHole:MountingHole_2.2mm_M2_Pad, F.Cu at (63.5, 201.6)
- added REF**: MountingHole_2.2mm_M2_Pad, MountingHole:MountingHole_2.2mm_M2_Pad, F.Cu at (192.1, 201.6)
- added REF**: MountingHole_2.2mm_M2_Pad, MountingHole:MountingHole_2.2mm_M2_Pad, F.Cu at (325.4, 192.1)
- added REF**: MountingHole_2.2mm_M2_Pad, MountingHole:MountingHole_2.2mm_M2_Pad, F.Cu at (325.4, 115.9)
- added REF**: MountingHole_2.2mm_M2_Pad, MountingHole:MountingHole_2.2mm_M2_Pad, F.Cu at (192.1, 115.9)
- added REF**: MountingHole_2.2mm_M2_Pad, MountingHole:MountingHole_2.2mm_M2_Pad, F.Cu at (58.7, 115.9)
- added REF**: MountingHole_2.2mm_M2_Pad, MountingHole:MountingHole_2.2mm_M2_Pad, F.Cu at (194.6, 93.0)
- added REF**: MountingHole_2.2mm_M2_Pad, MountingHole:MountingHole_2.2mm_M2_Pad, F.Cu at (194.6, 44.1)
- renumbered REF** to H_PLATE_BL, REF** to H_PLATE_BR, REF** to H_PLATE_TL, REF** to H_PLATE_TR

Commit message: hole labels
Parts:
- renumbered REF** to H_KEYS_BL, REF** to H_KEYS_BM, REF** to H_KEYS_BR, REF** to H_KEYS_TL, REF** to H_KEYS_TM, REF** to H_KEYS_TR, REF** to H_PLATE_MB, REF** to H_PLATE_TM
Changed lines of the file:
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@@
   (general
     (thickness 1.6)
-    (drawings 7)
+    (drawings 6)
     (tracks 0)
     (zones 0)
@@
     (tags "mounting hole 2.2mm m2")
     (attr virtual)
-    (fp_text reference REF** (at 0 -3.2) (layer F.SilkS)
+    (fp_text reference H_KEYS_BL (at 0 -3.2) (layer Cmts.User) hide
       (effects (font (size 1 1) (thickness 0.15)))
     )
@@
       (effects (font (size 1 1) (thickness 0.15)))
     )
-    (fp_text user %R (at 0.3 0) (layer F.Fab)
-      (effects (font (size 1 1) (thickness 0.15)))
-    )
     (fp_circle (center 0 0) (end 2.2 0) (layer Cmts.User) (width 0.15))
     (fp_circle (center 0 0) (end 2.45 0) (layer F.CrtYd) (width 0.05))
@@
     (tags "mounting hole 2.2mm m2")
     (attr virtual)
-    (fp_text reference REF** (at 0 -3.2) (layer F.SilkS)
+    (fp_text reference H_KEYS_BM (at 0 -3.2) (layer Cmts.User) hide
       (effects (font (size 1 1) (thickness 0.15)))
     )
@@
       (effects (font (size 1 1) (thickness 0.15)))
     )
-    (fp_text user %R (at 0.3 0) (layer F.Fab)
-      (effects (font (size 1 1) (thickness 0.15)))
-    )
     (fp_circle (center 0 0) (end 2.2 0) (layer Cmts.User) (width 0.15))
     (fp_circle (center 0 0) (end 2.45 0) (layer F.CrtYd) (width 0.05))
@@
     (tags "mounting hole 2.2mm m2")
     (attr virtual)
-    (fp_text reference REF** (at 0 -3.2) (layer F.SilkS)
+    (fp_text reference H_KEYS_BR (at 0 -3.2) (layer Cmts.User) hide
       (effects (font (size 1 1) (thickness 0.15)))
     )
@@
       (effects (font (size 1 1) (thickness 0.15)))
     )
-    (fp_text user %R (at 0.3 0) (layer F.Fab)
-      (effects (font (size 1 1) (thickness 0.15)))
-    )
     (fp_circle (center 0 0) (end 2.2 0) (layer Cmts.User) (width 0.15))
     (fp_circle (center 0 0) (end 2.45 0) (layer F.CrtYd) (width 0.05))
@@
     (tags "mounting hole 2.2mm m2")
     (attr virtual)
-    (fp_text reference REF** (at 0 -3.2) (layer F.SilkS)
+    (fp_text reference H_KEYS_TR (at 0 -3.2) (layer Cmts.User) hide
       (effects (font (size 1 1) (thickness 0.15)))
     )
@@
       (effects (font (size 1 1) (thickness 0.15)))
     )
-    (fp_text user %R (at 0.3 0) (layer F.Fab)
-      (effects (font (size 1 1) (thickness 0.15)))
-    )
     (fp_circle (center 0 0) (end 2.2 0) (layer Cmts.User) (width 0.15))
     (fp_circle (center 0 0) (end 2.45 0) (layer F.CrtYd) (width 0.05))
@@
     (tags "mounting hole 2.2mm m2")
     (attr virtual)
-    (fp_text reference REF** (at 0 -3.2) (layer F.SilkS)
+    (fp_text reference H_KEYS_TM (at 0 -3.2) (layer Cmts.User) hide
       (effects (font (size 1 1) (thickness 0.15)))
     )
@@
       (effects (font (size 1 1) (thickness 0.15)))
     )
-    (fp_text user %R (at 0.3 0) (layer F.Fab)
-      (effects (font (size 1 1) (thickness 0.15)))
-    )
     (fp_circle (center 0 0) (end 2.2 0) (layer Cmts.User) (width 0.15))
     (fp_circle (center 0 0) (end 2.45 0) (layer F.CrtYd) (width 0.05))
@@
     (tags "mounting hole 2.2mm m2")
     (attr virtual)
-    (fp_text reference REF** (at 0 -3.2) (layer F.SilkS)
+    (fp_text reference H_KEYS_TL (at 0 -3.2) (layer Cmts.User) hide
       (effects (font (size 1 1) (thickness 0.15)))
     )
@@
       (effects (font (size 1 1) (thickness 0.15)))
     )
-    (fp_text user %R (at 0.3 0) (layer F.Fab)
-      (effects (font (size 1 1) (thickness 0.15)))
-    )
     (fp_circle (center 0 0) (end 2.2 0) (layer Cmts.User) (width 0.15))
     (fp_circle (center 0 0) (end 2.45 0) (layer F.CrtYd) (width 0.05))
@@
     (tags "mounting hole 2.2mm m2")
     (attr virtual)
-    (fp_text reference REF** (at 0 -3.2) (layer F.SilkS)
+    (fp_text reference H_PLATE_MB (at 0 -3.2) (layer Cmts.User) hide
       (effects (font (size 1 1) (thickness 0.15)))
     )
@@
       (effects (font (size 1 1) (thickness 0.15)))
     )
-    (fp_text user %R (at 0.3 0) (layer F.Fab)
-      (effects (font (size 1 1) (thickness 0.15)))
-    )
     (fp_circle (center 0 0) (end 2.2 0) (layer Cmts.User) (width 0.15))
     (fp_circle (center 0 0) (end 2.45 0) (layer F.CrtYd) (width 0.05))
@@
     (tags "mounting hole 2.2mm m2")
     (attr virtual)
-    (fp_text reference REF** (at 0 -3.2) (layer F.SilkS)
+    (fp_text reference H_PLATE_TM (at 0 -3.2) (layer Cmts.User) hide
       (effects (font (size 1 1) (thickness 0.15)))
     )
@@
       (effects (font (size 1 1) (thickness 0.15)))
     )
-    (fp_text user %R (at 0.3 0) (layer F.Fab)
-      (effects (font (size 1 1) (thickness 0.15)))
-    )
     (fp_circle (center 0 0) (end 2.2 0) (layer Cmts.User) (width 0.15))
     (fp_circle (center 0 0) (end 2.45 0) (layer F.CrtYd) (width 0.05))
@@
   (gr_line (start 39.6875 40.3225) (end 39.6875 211.1375) (layer Edge.Cuts) (width 0.15))
   (gr_line (start 39.6875 40.3225) (end 344.4875 40.3225) (layer Edge.Cuts) (width 0.15))
-  (gr_line (start 43.4975 93.0275) (end 340.6775 93.0275) (layer Dwgs.User) (width 0.15))
   (gr_text "By 001" (at 332.6875 57.8375) (layer F.SilkS)
     (effects (font (size 2 1.5) (thickness 0.2)))
