File: pcb/00Key.kicad_pcb (KiCad board)
At the start: 2 copper layers, 304.8 x 170.8 mm, 268 parts, among them Q1 IRLZ44N, U1 Teensy4.1

Commit message: traces
Routing:
- net LEDGND: track 0.00 -> 1690.6 mm
- net col0: track 0.00 -> 392.2 mm
- net 5V: track 0.00 -> 384.0 mm
- net col1: track 0.00 -> 383.8 mm
- net col3: track 0.00 -> 336.7 mm
- net col2: track 0.00 -> 335.8 mm
- net row0: track 0.00 -> 333.5 mm
- net row1: track 0.00 -> 313.9 mm
- net row2: track 0.00 -> 306.5 mm
- net GND: track 0.00 -> 300.1 mm
- net row3: track 0.00 -> 299.1 mm
- net col4: track 0.00 -> 287.1 mm
- net row4: track 0.00 -> 285.2 mm
- net row5: track 0.00 -> 279.1 mm
- net col5: track 0.00 -> 273.5 mm, vias 0 -> 1
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