File: pcb/kicad/00Key.kicad_pcb (KiCad board)
At the start: 2 copper layers, 304.8 x 170.8 mm, 268 parts, among them Q1 IRLZ44N, U1 Teensy4.1

Commit message: lets just include the backup files
Other:
- net class Default removed
